File: eagle/808_handclap.sch (EAGLE design)
At the start: 94 parts, among them IC1 LM339N, IC2 TL072P, IC3 TL072P, Q28 BC546, Q29 BC556, Q35 BC546, Q69 BC546, Q70 BC546, Q71 BC556, Q72 BC556, Q73 BC546, U1 POWER, U22 BA6110SIL

Commit message: starting over from yocto
Parts:
- removed ACCENT, OUT, TRIG: LSP10, solpad:LSP10
- removed C1: 0.1, TR808clone:C-EU050-024X044
- removed C29: 47/16, TR808clone:CPOL-EUE2.5-5
- removed C31: 1/50, TR808clone:CPOL-EUE2.5-5
- removed D1: 1N4148DO35-7, TR808clone:1N4148DO35-7
- removed IC1: LM339N, linear:LM339N
- removed IC2, IC3: TL072P, linear:TL072P
- removed LEVEL: 100K(A), pot:3RP/1610N
- removed Q28, Q35, Q69, Q70, Q73: BC546, transistor:BC546-NPN-TO92-CBE
- removed Q29: BC556, transistor:BC556B-PNP-TO92-EBC
- removed Q71, Q72: BC556, transistor:BC556A-PNP-TO92-EBC
- removed R1: 100K, TR808clone:R-EU_0207/2V
- removed R124: 100R, TR808clone:R-EU_0207/5V
- removed R127: 4K7, TR808clone:R-EU_0207/7
- removed R128, R130: 1M, TR808clone:R-EU_0207/7
- removed R129: 330K, TR808clone:R-EU_0207/7
- removed R131: 300K, TR808clone:R-EU_0207/5V
- removed TM4: 22KB, TR808clone:TRIM_EU-CT6
- added OUTPUT, WHITE_NOISE: AUDIO-JACK, erthenvar:AUDIO-JACK
- added Q1, Q3, Q4: 2N3906, transistor-pnp:2N3906
- added Q2, Q5, Q6, Q7: 2N3904, transistor-npn:2N3904
- added R200': 10K, TR808clone:R-EU_0207/5V
- added U19, U21: µPC4558C, TR808clone:µPC4558C
- added U23: AN6912, TR808clone:AN6912
- added VR17: 100K(A), pot:3RP/1610N
- added WHITE_NORM: 22-23-2021, con-molex:22-23-2021
- C127, C128, C129, C139, C152: device TR808clone:C-EU050-025X075 -> TR808clone:C-EU3.5MM_PITCH
- C136, C137, C138: device TR808clone:C-EU050-025X075 -> TR808clone:C-EU050-024X044
- C140: value 2n7 -> 27n; device TR808clone:C-EU050-025X075 -> TR808clone:C-EU050-024X044
- C142: device TR808clone:C-EU050-025X075 -> TR808clone:C-EU025-025X050
- C145: device TR808clone:CPOL-EUE2,5-6E -> TR808clone:CPOL-EUE2-5
- C146: device TR808clone:C-EU050-025X075 -> TR808clone:C-EU4MM_PITCH
- R103, R104, R105, R106, R332, R333, R348, R349, R350, R351, R352, R353, R354, R356, R357, R358, R359, R360, R361, R362, R363, R364, R366, R367, R368, R369, R370, R371, R372, R373, R374, R376, R378, R381, R382, R383: device TR808clone:R-EU_0207/7 -> TR808clone:R-EU_0207/5V
- R334: value 100K -> 150K; device TR808clone:R-EU_0207/7 -> TR808clone:R-EU_0207/2V
- R346: device TR808clone:R-EU_0207/7 -> TR808clone:R-EU_0207/2V
- R355: device TR808clone:R-EU_0309/10 -> TR808clone:R-EU_0207/5V
- R375: device TR808clone:R-EU_0207/2V -> TR808clone:R-EU_0207/5V
Connections:
- removed net CPTRIG: Q29.C, Q69.B, R360.1
- removed net CP_MA_OUT: OUT.MP, R296.1
- removed net N$38: Q28.C, R106.1
- removed net N$5: C1.1, D1.C, R1.2
- removed net N$693: R129.1, R130.2, TM4.S
- removed net N$694: IC2B.-IN, R129.2
- removed net N$695: C31.+, Q35.E, R128.1
- removed net N$696: C29.+, R124.1, R128.2
- removed net N$699: R127.2, TM4.A
- removed net N$700: C31.-, IC2B.+IN, R131.1
- new net +B7: U19G$3.V+, U21G$3.V+
- new net -B7: U19G$3.V-
- new net -B8: U23G$5.V-
- new net N$2: WHITE_NOISE.NORM, WHITE_NORM-1.S
- new net N$3: Q5.C, R106.1
- new net N$43: Q2.B, Q3.C, R360.1
- net +12V: now also Q2.C; no longer IC2P.V+, IC3P.V+, Q69.C, R124.2
- net -12V: now also Q4.C, Q7.E, R200'.2; no longer IC1P.GND, IC2P.V-, IC3P.V-, Q71.C, Q73.E
- net CP: now also U1.GATE; no longer C1.2
- net GND: now also OUTPUT.RING, Q5.E, U21B.+IN, U23G$5.V+, WHITE_NOISE.RING, WHITE_NORM-2.S; no longer C29.-, IC1P.V+, IC2A.+IN, Q28.E, Q35.B, R1.1, R127.1, R131.2, U22.P$3
- net N$1: now also OUTPUT.TIP, R296.1; no longer D1.A, TRIG.MP
- net N$10: now also U21B.OUT; no longer IC2A.OUT
- net N$37: now also Q3.B; no longer Q29.B
- net N$4: now also Q5.B; no longer Q28.B
- net N$40: now also Q6.B; no longer Q70.B
- net N$42: now also Q6.E, R200'.1; no longer Q70.E
- net N$44: now also Q2.E; no longer Q69.E
- net N$46: now also Q6.C; no longer Q70.C
- net N$48: now also Q4.B; no longer Q71.B
- net N$51: now also U23G$4.OUT; no longer IC1A.OUT
- net N$54: now also U21B.-IN; no longer IC2A.-IN
- net N$64: now also U23G$2.-IN, U23G$4.+IN; no longer IC1A.+IN, IC1B.-IN
- net N$66: now also Q1.B; no longer Q72.B
- net N$67: now also Q1.E, Q4.E; no longer Q71.E, Q72.E
- net N$68: now also U23G$2.OUT, U23G$4.-IN; no longer IC1A.-IN, IC1B.OUT
- net N$69: now also Q1.C; no longer Q72.C
- net N$70: now also Q7.C; no longer Q73.C
- net N$71: now also U23G$3.+IN; no longer IC1C.+IN
- net N$72: now also U23G$1.+IN; no longer IC1D.+IN
- net N$73: now also U23G$1.-IN; no longer IC1D.-IN
- net N$74: now also U23G$3.-IN; no longer IC1C.-IN
- net N$75: now also Q7.B; no longer Q73.B
- net N$77: now also U23G$2.+IN, U23G$3.OUT; no longer IC1B.+IN, IC1C.OUT
- net N$78: now also U23G$1.OUT; no longer IC1D.OUT
- net N$91: now also U19B.+IN; no longer IC3A.+IN
- net N$92: now also U19B.-IN, VR17.A; no longer IC3A.-IN, LEVEL.A
- net N$95: now also VR17.S; no longer LEVEL.S
- net N$97: now also U19B.OUT; no longer IC3A.OUT
- net TRIG: now also Q3.E, U1.CV; no longer ACCENT.MP, Q29.E
- net WN: now also WHITE_NOISE.TIP; no longer IC2B.OUT, R130.1
Other:
- note removed: "Noise"
- moved on the sheet: C127, C128, C129, C136, C137, C138, C139, C140, C141, C142, C143, C144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

Commit message: lm339
Parts:
- removed U23: AN6912, TR808clone:AN6912
- added IC1: LM339N, linear:LM339N
- TM3: device TR808clone:TRIM_EU-CT6 -> pot:TRIM_1234-S64YW
Connections:
- removed net -B8: U23G$5.V-
- net -12V: now also IC1P.GND
- net GND: now also IC1P.V+; no longer U23G$5.V+
- net N$51: now also IC1D.OUT; no longer U23G$4.OUT
- net N$64: now also IC1B.-IN, IC1D.+IN; no longer U23G$2.-IN, U23G$4.+IN
- net N$68: now also IC1B.OUT, IC1D.-IN; no longer U23G$2.OUT, U23G$4.-IN
- net N$71: now also IC1C.+IN; no longer U23G$3.+IN
- net N$72: now also IC1A.+IN; no longer U23G$1.+IN
- net N$73: now also IC1A.-IN; no longer U23G$1.-IN
- net N$74: now also IC1C.-IN; no longer U23G$3.-IN
- net N$77: now also IC1B.+IN, IC1C.OUT; no longer U23G$2.+IN, U23G$3.OUT
- net N$78: now also IC1A.OUT; no longer U23G$1.OUT

Commit message: opamps
Parts:
- removed U19, U21: µPC4558C, TR808clone:µPC4558C
- added IC2, IC3: TL071P, 808_lt:TL071P
Connections:
- removed net +B7: U19G$3.V+, U21G$3.V+
- removed net -B7: U19G$3.V-
- net +12V: now also IC2.V+, IC3.V+
- net -12V: now also IC2.V-, IC3.V-
- net GND: now also IC2.+IN; no longer U21B.+IN
- net N$10: now also IC2.OUT; no longer U21B.OUT
- net N$54: now also IC2.-IN; no longer U21B.-IN
- net N$91: now also IC3.+IN; no longer U19B.+IN
- net N$92: now also IC3.-IN; no longer U19B.-IN
- net N$97: now also IC3.OUT; no longer U19B.OUT
Other:
- moved on the sheet: R334

Commit message: pretty up schemo
Connections:
- removed net +5V: U1.+5V
Other:
- moved on the sheet: C127, C128, C129, C136, C137, C138, C139, C140, C141, C142, C143, C144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

Commit message: variable reverb mod
Parts:
- removed R376: 47K, TR808clone:R-EU_0207/5V
- added REVERB: 100k, pot:3RP/1610N
- C140: value 27n -> 2n7
Connections:
- net N$57: now also REVERB.E; no longer R376.1
- net N$92: now also REVERB.S; no longer R376.2
Other:
- moved on the sheet: C137, D68, D69
Changed lines of the file:
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@@
 <part name="GND21" library="supply1" deviceset="GND" device=""/>
 <part name="C152" library="TR808clone" deviceset="C-EU" device="3.5MM_PITCH" value="4.7n"/>
-<part name="R376" library="TR808clone" deviceset="R-EU_" device="0207/5V" value="47K"/>
 <part name="R346" library="TR808clone" deviceset="R-EU_" device="0207/2V" value="680"/>
 <part name="R342" library="TR808clone" deviceset="R-EU_" device="0207/7" value="15K"/>
@@
 <part name="R351" library="TR808clone" deviceset="R-EU_" device="0207/5V" value="4K7"/>
 <part name="R350" library="TR808clone" deviceset="R-EU_" device="0207/5V" value="1M"/>
-<part name="C140" library="TR808clone" deviceset="C-EU" device="050-024X044" value="27n"/>
+<part name="C140" library="TR808clone" deviceset="C-EU" device="050-024X044" value="2n7"/>
 <part name="D70" library="TR808clone" deviceset="1N4148" device="DO35-7"/>
 <part name="GND38" library="supply1" deviceset="GND" device=""/>
@@
 <part name="P-11" library="supply1" deviceset="-12V" device=""/>
 <part name="P-12" library="supply1" deviceset="-12V" device=""/>
+<part name="REVERB" library="pot" deviceset="3RP/1610N" device="" value="100k"/>
 </parts>
 <sheets>
@@
 <instance part="GND15" gate="1" x="43.18" y="116.84" rot="MR0"/>
 <instance part="GND16" gate="1" x="33.02" y="116.84" rot="MR0"/>
-<instance part="D69" gate="G$1" x="58.42" y="104.14" smashed="yes">
-<attribute name="NAME" x="55.88" y="100.8126" size="1.778" layer="95"/>
-</instance>
-<instance part="D68" gate="G$1" x="58.42" y="91.44" smashed="yes">
-<attribute name="NAME" x="55.88" y="93.1926" size="1.778" layer="95"/>
+<instance part="D69" gate="G$1" x="60.96" y="104.14" smashed="yes">
+<attribute name="NAME" x="58.42" y="100.8126" size="1.778" layer="95"/>
+</instance>
+<instance part="D68" gate="G$1" x="60.96" y="91.44" smashed="yes">
+<attribute name="NAME" x="58.42" y="93.1926" size="1.778" layer="95"/>
 </instance>
 <instance part="C139" gate="G$1" x="68.58" y="99.06" smashed="yes" rot="R180">
@@
 <instance part="R369" gate="G$1" x="93.98" y="106.68" rot="MR270"/>
 <instance part="R363" gate="G$1" x="93.98" y="132.08" rot="MR270"/>
-<instance part="C137" gate="G$1" x="86.36" y="132.08" smashed="yes">
-<attribute name="NAME" x="84.074" y="133.731" size="1.778" layer="95" rot="R180"/>
-<attribute name="VALUE" x="84.074" y="131.191" size="1.778" layer="96" rot="R180"/>
+<instance part="C137" gate="G$1" x="86.36" y="137.16" smashed="yes">
+<attribute name="NAME" x="84.074" y="138.811" size="1.778" layer="95" rot="R180"/>
+<attribute name="VALUE" x="84.074" y="136.271" size="1.778" layer="96" rot="R180"/>
 </instance>
 <instance part="TM3" gate="1" x="78.74" y="106.68" smashed="yes">
@@
 <attribute name="VALUE" x="109.474" y="105.791" size="1.778" layer="96" rot="R180"/>
 </instance>
-<instance part="R376" gate="G$1" x="111.76" y="96.52" rot="MR270"/>
 <instance part="R346" gate="G$1" x="106.68" y="139.7" rot="MR90"/>
 <instance part="R342" gate="G$1" x="119.38" y="144.78" rot="MR0"/>
@@
 <instance part="P-11" gate="1" x="149.86" y="137.16" rot="R180"/>
 <instance part="P-12" gate="1" x="208.28" y="86.36" rot="R180"/>
+<instance part="REVERB" gate="G$1" x="106.68" y="91.44"/>
 </instances>
 <busses>
@@
 <wire x1="88.9" y1="121.92" x2="86.36" y2="121.92" width="0.1524" layer="91"/>
 <pinref part="C137" gate="G$1" pin="2"/>
-<wire x1="86.36" y1="121.92" x2="86.36" y2="127" width="0.1524" layer="91"/>
+<wire x1="86.36" y1="121.92" x2="86.36" y2="132.08" width="0.1524" layer="91"/>
 <junction x="86.36" y="121.92"/>
 <pinref part="Q6" gate="G1" pin="B"/>
@@
 <wire x1="68.58" y1="109.22" x2="68.58" y2="104.14" width="0.1524" layer="91"/>
 <pinref part="D69" gate="G$1" pin="C"/>
-<wire x1="60.96" y1="104.14" x2="68.58" y2="104.14" width="0.1524" layer="91"/>
+<wire x1="63.5" y1="104.14" x2="68.58" y2="104.14" width="0.1524" layer="91"/>
 <junction x="68.58" y="104.14"/>
 </segment>
@@
 <pinref part="D68" gate="G$1" pin="A"/>
 <wire x1="53.34" y1="104.14" x2="53.34" y2="91.44" width="0.1524" layer="91"/>
-<wire x1="53.34" y1="91.44" x2="55.88" y2="91.44" width="0.1524" layer="91"/>
+<wire x1="53.34" y1="91.44" x2="58.42" y2="91.44" width="0.1524" layer="91"/>
 <pinref part="D69" gate="G$1" pin="A"/>
-<wire x1="55.88" y1="104.14" x2="53.34" y2="104.14" width="0.1524" layer="91"/>
+<wire x1="58.42" y1="104.14" x2="53.34" y2="104.14" width="0.1524" layer="91"/>
 <junction x="53.34" y="104.14"/>
 <pinref part="Q2" gate="G1" pin="E"/>
@@
 <pinref part="D68" gate="G$1" pin="C"/>
 <pinref part="R362" gate="G$1" pin="2"/>
-<wire x1="60.96" y1="91.44" x2="68.58" y2="91.44" width="0.1524" layer="91"/>
+<wire x1="63.5" y1="91.44" x2="68.58" y2="91.44" width="0.1524" layer="91"/>
 <pinref part="C143" gate="G$1" pin="+"/>
 <wire x1="76.2" y1="91.44" x2="68.58" y2="91.44" width="0.1524" layer="91"/>
@@
 <segment>
 <pinref part="C137" gate="G$1" pin="1"/>
-<wire x1="86.36" y1="134.62" x2="86.36" y2="144.78" width="0.1524" layer="91"/>
+<wire x1="86.36" y1="139.7" x2="86.36" y2="144.78" width="0.1524" layer="91"/>
 <pinref part="R342" gate="G$1" pin="2"/>
 <wire x1="86.36" y1="144.78" x2="106.68" y2="144.78" width="0.1524" layer="91"/>
@@
 <net name="N$57" class="0">
 <segment>
-<pinref part="R376" gate="G$1" pin="1"/>
 <pinref part="C152" gate="G$1" pin="2"/>
+<pinref part="REVERB" gate="G$1" pin="E"/>
+<wire x1="106.68" y1="96.52" x2="111.76" y2="96.52" width="0.1524" layer="91"/>
+<wire x1="111.76" y1="96.52" x2="111.76" y2="101.6" width="0.1524" layer="91"/>
 </segment>
 </net>
@@
 <net name="N$92" class="3">
 <segment>
-<pinref part="R376" gate="G$1" pin="2"/>
 <wire x1="111.76" y1="91.44" x2="111.76" y2="83.82" width="0.1524" layer="91"/>
 <pinref part="R378" gate="G$1" pin="2"/>
@@
 <wire x1="203.2" y1="83.82" x2="203.2" y2="78.74" width="0.1524" layer="91"/>
 <junction x="203.2" y="83.82"/>
-</segment>
-</net>
+<pinref part="REVERB" gate="G$1" pin="S"/>
+</segment>
+</net>

Commit message: 88pct autorouted
Parts:
- R334, R346: device TR808clone:R-EU_0207/2V -> TR808clone:R-EU_0207/7
- R350, R356, R363, R364, R367, R371, R374, R381: device TR808clone:R-EU_0207/5V -> TR808clone:R-EU_0207/7
- R359, R360, R362, R373: device TR808clone:R-EU_0207/5V -> TR808clone:R-EU_0309/10
Connections:
- net N$51: now also IC1A.OUT; no longer IC1D.OUT
- net N$64: now also IC1A.+IN; no longer IC1D.+IN
- net N$68: now also IC1A.-IN; no longer IC1D.-IN
- net N$72: now also IC1D.+IN; no longer IC1A.+IN
- net N$73: now also IC1D.-IN; no longer IC1A.-IN
- net N$78: now also IC1D.OUT; no longer IC1A.OUT
Other:
- moved on the sheet: C150, IC1A, IC1D, R364, R371

Commit message: 88pct autorouted
Parts:
- R105: device TR808clone:R-EU_0207/5V -> TR808clone:R-EU_0207/2V
- R334: device TR808clone:R-EU_0207/7 -> TR808clone:R-EU_0309/10
Changed lines of the file:
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@@
 <part name="R104" library="TR808clone" deviceset="R-EU_" device="0207/5V" value="10K"/>
 <part name="R106" library="TR808clone" deviceset="R-EU_" device="0207/5V" value="10K"/>
-<part name="R105" library="TR808clone" deviceset="R-EU_" device="0207/5V" value="4K7"/>
+<part name="R105" library="TR808clone" deviceset="R-EU_" device="0207/2V" value="4K7"/>
 <part name="GND15" library="supply1" deviceset="GND" device=""/>
 <part name="GND16" library="supply1" deviceset="GND" device=""/>
@@
 <part name="C129" library="TR808clone" deviceset="C-EU" device="3.5MM_PITCH" value="4.7n"/>
 <part name="C128" library="TR808clone" deviceset="C-EU" device="3.5MM_PITCH" value="4.7n"/>
-<part name="R334" library="TR808clone" deviceset="R-EU_" device="0207/7" value="150K"/>
+<part name="R334" library="TR808clone" deviceset="R-EU_" device="0309/10" value="150K"/>
 <part name="R333" library="TR808clone" deviceset="R-EU_" device="0207/5V" value="10K"/>
 <part name="R332" library="TR808clone" deviceset="R-EU_" device="0207/5V" value="27K"/>
