File: eagle/808_handclap.sch (EAGLE design)
At the start: 82 parts, among them IC1 LM339N, IC2 TL071P, IC3 TL071P, Q1 2N3906, Q2 2N3904, Q3 2N3906, Q4 2N3906, Q5 2N3904, Q6 2N3904, Q7 2N3904, U1 POWER, U22 BA6110SIL

Commit message: more hand routes
Parts:
- C137: device TR808clone:C-EU050-024X044 -> TR808clone:C-EU075-032X103
- D70: value 1N4148DO35-10 -> 1N4148DO35-7; device TR808clone:1N4148DO35-10 -> TR808clone:1N4148DO35-7
- R296, R353, R356: device TR808clone:R-EU_0207/5V -> TR808clone:R-EU_0207/7
- R334: device TR808clone:R-EU_0309/10 -> TR808clone:R-EU_0207/7
Changed lines of the file:
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@@
 <part name="R369" library="TR808clone" deviceset="R-EU_" device="0207/2V" value="330R"/>
 <part name="R363" library="TR808clone" deviceset="R-EU_" device="0207/7" value="10K"/>
-<part name="C137" library="TR808clone" deviceset="C-EU" device="050-024X044" value="33n"/>
+<part name="C137" library="TR808clone" deviceset="C-EU" device="075-032X103" value="33n"/>
 <part name="TM3" library="pot" deviceset="TRIM_1234-" device="S64YW" value="10K(B)"/>
 <part name="GND20" library="supply1" deviceset="GND" device=""/>
@@
 <part name="C129" library="TR808clone" deviceset="C-EU" device="3.5MM_PITCH" value="4.7n"/>
 <part name="C128" library="TR808clone" deviceset="C-EU" device="3.5MM_PITCH" value="4.7n"/>
-<part name="R334" library="TR808clone" deviceset="R-EU_" device="0309/10" value="150K"/>
+<part name="R334" library="TR808clone" deviceset="R-EU_" device="0207/7" value="150K"/>
 <part name="R333" library="TR808clone" deviceset="R-EU_" device="0207/5V" value="10K"/>
 <part name="R332" library="TR808clone" deviceset="R-EU_" device="0207/7" value="27K"/>
@@
 <part name="GND33" library="supply1" deviceset="GND" device=""/>
 <part name="GND34" library="supply1" deviceset="GND" device=""/>
-<part name="R356" library="TR808clone" deviceset="R-EU_" device="0207/5V" value="1M"/>
+<part name="R356" library="TR808clone" deviceset="R-EU_" device="0207/7" value="1M"/>
 <part name="R355" library="TR808clone" deviceset="R-EU_" device="0207/5V" value="2K7"/>
 <part name="R354" library="TR808clone" deviceset="R-EU_" device="0207/5V" value="5K6"/>
 <part name="GND35" library="supply1" deviceset="GND" device=""/>
-<part name="R353" library="TR808clone" deviceset="R-EU_" device="0207/5V" value="4K7"/>
+<part name="R353" library="TR808clone" deviceset="R-EU_" device="0207/7" value="4K7"/>
 <part name="R352" library="TR808clone" deviceset="R-EU_" device="0309/10" value="4K7"/>
 <part name="GND36" library="supply1" deviceset="GND" device=""/>
@@
 <part name="R350" library="TR808clone" deviceset="R-EU_" device="0207/7" value="1M"/>
 <part name="C140" library="TR808clone" deviceset="C-EU" device="050-024X044" value="2n7"/>
-<part name="D70" library="TR808clone" deviceset="1N4148" device="DO35-10" value="1N4148DO35-10"/>
+<part name="D70" library="TR808clone" deviceset="1N4148" device="DO35-7" value="1N4148DO35-7"/>
 <part name="GND38" library="supply1" deviceset="GND" device=""/>
 <part name="GND39" library="supply1" deviceset="GND" device=""/>
@@
 <part name="C145" library="TR808clone" deviceset="CPOL-EU" device="E2-5" value="33/6.3"/>
 <part name="VR17" library="pot" deviceset="3RP/1610N" device="" value="100K(A)"/>
-<part name="R296" library="TR808clone" deviceset="R-EU_" device="0207/5V" value="1K"/>
+<part name="R296" library="TR808clone" deviceset="R-EU_" device="0207/7" value="1K"/>
 <part name="GND48" library="supply1" deviceset="GND" device=""/>
 <part name="U22" library="TR808clone" deviceset="BA6110" device="SIL"/>

Commit message: routed
Parts:
- C127: device TR808clone:C-EU3.5MM_PITCH -> TR808clone:C-EU075-032X103
- C145: device TR808clone:CPOL-EUE2-5 -> TR808clone:CPOL-EUE3.5-8
- C149: device TR808clone:C-EU025-025X050 -> TR808clone:C-EU050-024X044
- R103, R368: device TR808clone:R-EU_0207/5V -> TR808clone:R-EU_0207/7
- R105: device TR808clone:R-EU_0207/2V -> TR808clone:R-EU_0207/5V
- R369: device TR808clone:R-EU_0207/2V -> TR808clone:R-EU_0207/7
- R381, R382: device TR808clone:R-EU_0207/7 -> TR808clone:R-EU_0207/5V
Changed lines of the file:
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@@
 </classes>
 <parts>
-<part name="R103" library="TR808clone" deviceset="R-EU_" device="0207/5V" value="22K"/>
+<part name="R103" library="TR808clone" deviceset="R-EU_" device="0207/7" value="22K"/>
 <part name="R104" library="TR808clone" deviceset="R-EU_" device="0207/7" value="10K"/>
 <part name="R106" library="TR808clone" deviceset="R-EU_" device="0207/5V" value="10K"/>
-<part name="R105" library="TR808clone" deviceset="R-EU_" device="0207/2V" value="4K7"/>
+<part name="R105" library="TR808clone" deviceset="R-EU_" device="0207/5V" value="4K7"/>
 <part name="GND15" library="supply1" deviceset="GND" device=""/>
 <part name="GND16" library="supply1" deviceset="GND" device=""/>
@@
 <part name="R362" library="TR808clone" deviceset="R-EU_" device="0309/10" value="330K"/>
 <part name="R370" library="TR808clone" deviceset="R-EU_" device="0309/10" value="47K"/>
-<part name="R369" library="TR808clone" deviceset="R-EU_" device="0207/2V" value="330R"/>
+<part name="R369" library="TR808clone" deviceset="R-EU_" device="0207/7" value="330R"/>
 <part name="R363" library="TR808clone" deviceset="R-EU_" device="0207/7" value="10K"/>
 <part name="C137" library="TR808clone" deviceset="C-EU" device="075-032X103" value="33n"/>
@@
 <part name="R333" library="TR808clone" deviceset="R-EU_" device="0207/5V" value="10K"/>
 <part name="R332" library="TR808clone" deviceset="R-EU_" device="0207/7" value="27K"/>
-<part name="C127" library="TR808clone" deviceset="C-EU" device="3.5MM_PITCH" value="1.8n"/>
+<part name="C127" library="TR808clone" deviceset="C-EU" device="075-032X103" value="1.8n"/>
 <part name="C136" library="TR808clone" deviceset="C-EU" device="050-024X044" value="22n"/>
 <part name="R372" library="TR808clone" deviceset="R-EU_" device="0207/7" value="39K"/>
-<part name="R382" library="TR808clone" deviceset="R-EU_" device="0207/7" value="1K"/>
-<part name="R381" library="TR808clone" deviceset="R-EU_" device="0207/7" value="1K"/>
+<part name="R382" library="TR808clone" deviceset="R-EU_" device="0207/5V" value="1K"/>
+<part name="R381" library="TR808clone" deviceset="R-EU_" device="0207/5V" value="1K"/>
 <part name="C146" library="TR808clone" deviceset="C-EU" device="4MM_PITCH" value="18n"/>
 <part name="GND22" library="supply1" deviceset="GND" device=""/>
@@
 <part name="R366" library="TR808clone" deviceset="R-EU_" device="0207/7" value="15K"/>
 <part name="R364" library="TR808clone" deviceset="R-EU_" device="0309/10" value="2K2"/>
-<part name="R368" library="TR808clone" deviceset="R-EU_" device="0207/5V" value="470K"/>
+<part name="R368" library="TR808clone" deviceset="R-EU_" device="0207/7" value="470K"/>
 <part name="R371" library="TR808clone" deviceset="R-EU_" device="0207/7" value="15K"/>
 <part name="R367" library="TR808clone" deviceset="R-EU_" device="0207/7" value="330"/>
@@
 <part name="R373" library="TR808clone" deviceset="R-EU_" device="0207/7" value="47K"/>
 <part name="R375" library="TR808clone" deviceset="R-EU_" device="0207/5V" value="470K"/>
-<part name="C149" library="TR808clone" deviceset="C-EU" device="025-025X050" value="220p"/>
-<part name="C145" library="TR808clone" deviceset="CPOL-EU" device="E2-5" value="33/6.3"/>
+<part name="C149" library="TR808clone" deviceset="C-EU" device="050-024X044" value="220p"/>
+<part name="C145" library="TR808clone" deviceset="CPOL-EU" device="E3.5-8" value="33/6.3"/>
 <part name="VR17" library="pot" deviceset="3RP/1610N" device="" value="100K(A)"/>
 <part name="R296" library="TR808clone" deviceset="R-EU_" device="0207/7" value="1K"/>

Commit message: tweaks
Parts:
- R383: device TR808clone:R-EU_0207/2V -> TR808clone:R-EU_0207/7
Other:
- moved on the sheet: R374
Changed lines of the file:
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@@
 <part name="C150" library="TR808clone" deviceset="C-EU" device="3.5MM_PITCH" value="1n"/>
 <part name="R378" library="TR808clone" deviceset="R-EU_" device="0207/7" value="100K"/>
-<part name="R383" library="TR808clone" deviceset="R-EU_" device="0207/2V" value="82K"/>
+<part name="R383" library="TR808clone" deviceset="R-EU_" device="0207/7" value="82K"/>
 <part name="GND29" library="supply1" deviceset="GND" device=""/>
 <part name="R366" library="TR808clone" deviceset="R-EU_" device="0207/7" value="15K"/>
@@
 <instance part="GND26" gate="1" x="132.08" y="149.86" rot="MR0"/>
 <instance part="GND27" gate="1" x="106.68" y="132.08" rot="MR0"/>
-<instance part="R374" gate="G$1" x="144.78" y="88.9" rot="MR270"/>
+<instance part="R374" gate="G$1" x="144.78" y="91.44" rot="MR270"/>
 <instance part="C150" gate="G$1" x="185.42" y="101.6" smashed="yes">
 <attribute name="NAME" x="183.134" y="104.521" size="1.778" layer="95" rot="R180"/>
@@
 <segment>
 <pinref part="R374" gate="G$1" pin="2"/>
-<wire x1="144.78" y1="83.82" x2="147.32" y2="48.26" width="0.1524" layer="91"/>
+<wire x1="144.78" y1="86.36" x2="147.32" y2="48.26" width="0.1524" layer="91"/>
 <wire x1="147.32" y1="48.26" x2="154.94" y2="48.26" width="0.1524" layer="91"/>
 <pinref part="Q1" gate="G$1" pin="C"/>
@@
 <pinref part="U22" gate="G$1" pin="C"/>
 <pinref part="R374" gate="G$1" pin="1"/>
-<wire x1="146.05" y1="114.3" x2="144.78" y2="93.98" width="0.1524" layer="91"/>
-</segment>
-</net>
+<wire x1="146.05" y1="114.3" x2="144.78" y2="96.52" width="0.1524" layer="91"/>
+</segment>
+</net>
