File: eagle/808_handclap.brd (EAGLE design)
At the start: 100.8 x 81.8 mm, 82 parts, among them IC1 LM339N, IC2 TL071P, IC3 TL071P, Q1 2N3906, Q2 2N3904, Q3 2N3906, Q4 2N3906, Q5 2N3904, Q6 2N3904, Q7 2N3904, U1 POWER, U22 BA6110SIL

Commit message: changed c140 to 27n to make separate hits audible
Parts:
- C140: value 2n7 -> 27n
Changed lines of the file:
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@@
 <?xml version="1.0" encoding="utf-8"?>
 <!DOCTYPE eagle SYSTEM "eagle.dtd">
-<eagle version="7.2.0">
+<eagle version="7.1.0">
 <drawing>
 <settings>
@@
 <element name="C138" library="TR808clone" package="C050-024X044" value="47n" x="26.924" y="69.85" rot="R270"/>
 <element name="C139" library="TR808clone" package="C035-025X75" value="18n" x="33.02" y="67.31" rot="R270"/>
-<element name="C140" library="TR808clone" package="C050-024X044" value="2n7" x="49.53" y="17.78"/>
+<element name="C140" library="TR808clone" package="C050-024X044" value="27n" x="49.53" y="17.78"/>
 <element name="C141" library="TR808clone" package="C035-025X75" value="1n" x="86.36" y="16.51"/>
 <element name="C142" library="TR808clone" package="C050-025X075" value="220p" x="69.342" y="29.21"/>
